File: opilio_pcb/opilio3.kicad_sch (KiCad schematic)
At the start: 90 parts, among them J1 Screw_Terminal_01x02, J2 Conn_01x02_Male, J3 USB_B_Micro, J4 Program, Q1 HSBA3048, Q2 HSBA3048, U1 EUP3458, U2 SCT51240, U3 SCT51240, U4 USBLC6-2SC6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

Commit message: add power flag
Changed lines of the file:
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@@
     (pin "4")
+  )
+  (symbol (lib_id "power:PWR_FLAG") (at 136.017 69.596 0) (unit 1)
+    (in_bom yes) (on_board yes) (fields_autoplaced)
+    (property "Reference" "#FLG?" (id 0) (at 136.017 67.691 0)
+      (effects (font (size 1.27 1.27)) hide)
+    )
+    (property "Value" "PWR_FLAG" (id 1) (at 136.017 66.0202 0))
+    (property "Footprint" "" (id 2) (at 136.017 69.596 0)
+      (effects (font (size 1.27 1.27)) hide)
+    )
+    (property "Datasheet" "~" (id 3) (at 136.017 69.596 0)
+      (effects (font (size 1.27 1.27)) hide)
+    )
+    (pin "1")
   )
   (symbol (lib_id "power:GND") (at 168.91 35.306 270) (unit 1)
@@
   )
   (symbol_instances
+    (path "/a78f4701-09c7-499d-a431-c3099a155bf7"
+      (reference "#FLG?") (unit 1) (value "PWR_FLAG") (footprint "")
+    )
     (path "/c1e1ecb3-dd47-40fa-886f-0d9dd05b0e48"
       (reference "#PWR01") (unit 1) (value "+3.3V") (footprint "")

Commit message: save standby
Connections:
- net +3V3 renamed +3.3V
Changed lines of the file:
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@@
   (symbol (lib_id "power:PWR_FLAG") (at 136.017 69.596 0) (unit 1)
     (in_bom yes) (on_board yes) (fields_autoplaced)
-    (property "Reference" "#FLG?" (id 0) (at 136.017 67.691 0)
+    (property "Reference" "#FLG0101" (id 0) (at 136.017 67.691 0)
       (effects (font (size 1.27 1.27)) hide)
     )
@@
     (pin "1")
     (pin "2")
+  )
+  (symbol (lib_id "power:PWR_FLAG") (at 124.587 24.257 0) (unit 1)
+    (in_bom yes) (on_board yes)
+    (property "Reference" "#FLG0102" (id 0) (at 124.587 22.352 0)
+      (effects (font (size 1.27 1.27)) hide)
+    )
+    (property "Value" "PWR_FLAG" (id 1) (at 122.555 20.701 0))
+    (property "Footprint" "" (id 2) (at 124.587 24.257 0)
+      (effects (font (size 1.27 1.27)) hide)
+    )
+    (property "Datasheet" "~" (id 3) (at 124.587 24.257 0)
+      (effects (font (size 1.27 1.27)) hide)
+    )
+    (pin "1")
   )
   (symbol (lib_id "power:GND") (at 63.119 27.686 0) (unit 1)
@@
   (symbol_instances
     (path "/a78f4701-09c7-499d-a431-c3099a155bf7"
-      (reference "#FLG?") (unit 1) (value "PWR_FLAG") (footprint "")
+      (reference "#FLG0101") (unit 1) (value "PWR_FLAG") (footprint "")
+    )
+    (path "/e8e3e2e3-7ac9-4535-9ead-c94eb0116dc6"
+      (reference "#FLG0102") (unit 1) (value "PWR_FLAG") (footprint "")
     )
     (path "/c1e1ecb3-dd47-40fa-886f-0d9dd05b0e48"

Commit message: update pcb
Parts:
- C16, C17, C23, C24: value 100nF -> 10nF
- R10, R15, R3, R9: value 4k7 -> 10k
- R2: value 10k -> 22R
Changed lines of the file:
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@@
       (effects (font (size 1.27 1.27)) (justify left))
     )
-    (property "Value" "100nF" (id 1) (at 241.3 96.266 90)
+    (property "Value" "10nF" (id 1) (at 241.3 96.266 90)
       (effects (font (size 1.27 1.27)) (justify left))
     )
@@
       (effects (font (size 1.27 1.27)) (justify left))
     )
-    (property "Value" "10k" (id 1) (at 64.897 26.035 0)
+    (property "Value" "22R" (id 1) (at 64.897 26.035 0)
       (effects (font (size 1.27 1.27)) (justify left))
     )
@@
     (in_bom yes) (on_board yes)
     (property "Reference" "R9" (id 0) (at 238.252 83.947 90))
-    (property "Value" "4k7" (id 1) (at 238.252 89.027 90))
+    (property "Value" "10k" (id 1) (at 238.252 89.027 90))
     (property "Footprint" "Resistor_SMD:R_0603_1608Metric_Pad0.98x0.95mm_HandSolder" (id 2) (at 238.252 86.487 0)
       (effects (font (size 1.27 1.27)) hide)
@@
     (in_bom yes) (on_board yes)
     (property "Reference" "R10" (id 0) (at 196.596 83.947 90))
-    (property "Value" "4k7" (id 1) (at 196.596 89.027 90))
+    (property "Value" "10k" (id 1) (at 196.596 89.027 90))
     (property "Footprint" "Resistor_SMD:R_0603_1608Metric_Pad0.98x0.95mm_HandSolder" (id 2) (at 196.596 86.487 0)
       (effects (font (size 1.27 1.27)) hide)
@@
     (in_bom yes) (on_board yes)
     (property "Reference" "R3" (id 0) (at 259.461 26.416 90))
-    (property "Value" "4k7" (id 1) (at 259.461 31.496 90))
+    (property "Value" "10k" (id 1) (at 259.461 31.496 90))
     (property "Footprint" "Resistor_SMD:R_0603_1608Metric_Pad0.98x0.95mm_HandSolder" (id 2) (at 259.461 28.956 0)
       (effects (font (size 1.27 1.27)) hide)
@@
     (in_bom yes) (on_board yes)
     (property "Reference" "R15" (id 0) (at 251.333 131.318 90))
-    (property "Value" "4k7" (id 1) (at 251.333 136.398 90))
+    (property "Value" "10k" (id 1) (at 251.333 136.398 90))
     (property "Footprint" "Resistor_SMD:R_0603_1608Metric_Pad0.98x0.95mm_HandSolder" (id 2) (at 251.333 133.858 0)
       (effects (font (size 1.27 1.27)) hide)
@@
       (effects (font (size 1.27 1.27)) (justify left))
     )
-    (property "Value" "100nF" (id 1) (at 254.381 143.637 90)
+    (property "Value" "10nF" (id 1) (at 254.381 143.637 90)
       (effects (font (size 1.27 1.27)) (justify left))
     )
@@
       (effects (font (size 1.27 1.27)) (justify left))
     )
-    (property "Value" "100nF" (id 1) (at 199.644 96.266 90)
+    (property "Value" "10nF" (id 1) (at 199.644 96.266 90)
       (effects (font (size 1.27 1.27)) (justify left))
     )
@@
       (effects (font (size 1.27 1.27)) (justify left))
     )
-    (property "Value" "100nF" (id 1) (at 262.509 38.735 90)
+    (property "Value" "10nF" (id 1) (at 262.509 38.735 90)
       (effects (font (size 1.27 1.27)) (justify left))
     )
@@
     )
     (path "/20a7523c-fe7d-4f2a-8c01-4eeb876f876c"
-      (reference "C16") (unit 1) (value "100nF") (footprint "Capacitor_SMD:C_0603_1608Metric_Pad1.08x0.95mm_HandSolder")
+      (reference "C16") (unit 1) (value "10nF") (footprint "Capacitor_SMD:C_0603_1608Metric_Pad1.08x0.95mm_HandSolder")
     )
     (path "/8d6eb2b3-dee9-410b-9b93-60e729b51ca6"
-      (reference "C17") (unit 1) (value "100nF") (footprint "Capacitor_SMD:C_0603_1608Metric_Pad1.08x0.95mm_HandSolder")
+      (reference "C17") (unit 1) (value "10nF") (footprint "Capacitor_SMD:C_0603_1608Metric_Pad1.08x0.95mm_HandSolder")
     )
     (path "/4796091b-eee0-468d-ae28-3df6a250e484"
@@
     )
     (path "/7a4e94b6-f587-4a19-a8b6-20539b6555cb"
-      (reference "C23") (unit 1) (value "100nF") (footprint "Capacitor_SMD:C_0603_1608Metric_Pad1.08x0.95mm_HandSolder")
+      (reference "C23") (unit 1) (value "10nF") (footprint "Capacitor_SMD:C_0603_1608Metric_Pad1.08x0.95mm_HandSolder")
     )
     (path "/f9a43796-c8f7-4e92-a0e4-0ff2e0d684fe"
-      (reference "C24") (unit 1) (value "100nF") (footprint "Capacitor_SMD:C_0603_1608Metric_Pad1.08x0.95mm_HandSolder")
+      (reference "C24") (unit 1) (value "10nF") (footprint "Capacitor_SMD:C_0603_1608Metric_Pad1.08x0.95mm_HandSolder")
     )
     (path "/a113ab45-c224-45cf-9cff-14a460bb8ef8"
@@
     )
     (path "/473255dc-8035-43f0-b1fd-60d68bf17542"
-      (reference "R2") (unit 1) (value "10k") (footprint "Resistor_SMD:R_0603_1608Metric_Pad0.98x0.95mm_HandSolder")
+      (reference "R2") (unit 1) (value "22R") (footprint "Resistor_SMD:R_0603_1608Metric_Pad0.98x0.95mm_HandSolder")
     )
     (path "/4e3e959e-b2af-4986-8e2c-e2e74e7ae0db"
-      (reference "R3") (unit 1) (value "4k7") (footprint "Resistor_SMD:R_0603_1608Metric_Pad0.98x0.95mm_HandSolder")
+      (reference "R3") (unit 1) (value "10k") (footprint "Resistor_SMD:R_0603_1608Metric_Pad0.98x0.95mm_HandSolder")
     )
     (path "/7bb08001-7e60-4e0a-b06b-a44734cacf0c"
@@
     )
     (path "/48640d49-ea36-4a8c-a2c5-d5d52d8aaa99"
-      (reference "R9") (unit 1) (value "4k7") (footprint "Resistor_SMD:R_0603_1608Metric_Pad0.98x0.95mm_HandSolder")
+      (reference "R9") (unit 1) (value "10k") (footprint "Resistor_SMD:R_0603_1608Metric_Pad0.98x0.95mm_HandSolder")
     )
     (path "/4de7545d-6b1d-480b-a9c2-29e71c899d71"
-      (reference "R10") (unit 1) (value "4k7") (footprint "Resistor_SMD:R_0603_1608Metric_Pad0.98x0.95mm_HandSolder")
+      (reference "R10") (unit 1) (value "10k") (footprint "Resistor_SMD:R_0603_1608Metric_Pad0.98x0.95mm_HandSolder")
     )
     (path "/c8fa8fa3-be95-4a0c-bb19-a1e338cef170"
@@
     )
     (path "/56ec5d54-a989-4bfb-999d-5d1f48e5a1a1"
-      (reference "R15") (unit 1) (value "4k7") (footprint "Resistor_SMD:R_0603_1608Metric_Pad0.98x0.95mm_HandSolder")
+      (reference "R15") (unit 1) (value "10k") (footprint "Resistor_SMD:R_0603_1608Metric_Pad0.98x0.95mm_HandSolder")
     )
     (path "/151dbe14-095c-413c-9193-8601b139b4d6"
