File: opilio_pcb/v3.1/opilio3.1.kicad_pcb (KiCad board)
At the start: 4 copper layers, 80 x 40 mm, 87 parts, among them J1 Screw_Terminal_01x02, J2 Conn_01x02_Male, J3 USB_B_Micro, J4 Program, J5 Conn_01x02_Male, Q1 HSBA3048, Q2 HSBA3048, U1 AMS1117-3.3, U2 SCT51240, U3 SCT51240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

Commit message: moved opilio 3.1
Parts:
- added D10: B5819W, Diode_SMD:D_SOD-123, F.Cu at (157.2, 124.8)
- added D9: B5819W, Diode_SMD:D_SOD-123, F.Cu at (161.9, 128.6)
- moved C5 1.18 mm to (162.0, 125.1)
- moved C1 1.18 mm to (168.7, 122.7)
- moved F1 1.18 mm to (166.9, 127.9)
- moved FB1 1.18 mm to (166.9, 125.4)
- moved U1 1.18 mm to (163.1, 119.6)
Connections:
- F1 pad 1: +12V -> Net-(F1-Pad1)
Routing:
- net +5V: track 7.94 -> 29.2 mm, vias 0 -> 2
- net Net-(F1-Pad1): track 0.00 -> 9.00 mm
- net +12V: track 27.4 -> 31.1 mm
- net PUMP_EN: track 32.4 -> 31.6 mm
- net GND: track 111.0 -> 111.6 mm

Commit message: almost ready for v3.1
Parts:
- added G***: LOGO, LOGO, F.Cu at (152.7, 119.4)
- added G***: LOGO, LOGO, F.Cu at (128.0, 126.7)
- moved C24 1.69 mm to (139.8, 129.8)
- moved R3 1.55 mm to (139.8, 131.4)
- moved D10 0.91 mm to (158.1, 125.0)
Routing:
- net +5V: track 29.2 -> 33.6 mm
- net GND: track 111.6 -> 107.3 mm, vias 39 -> 70
- net FAN_GND: track 37.0 -> 39.9 mm, vias 12 -> 14
- net +12VF(F): track 108.7 -> 111.2 mm
- net +12V: track 31.1 -> 29.3 mm
- net Net-(D10-Pad1): track 9.00 -> 10.7 mm
- net PUMP_EN: track 31.6 -> 30.8 mm
- net +3.3V: track 50.0 -> 49.9 mm, vias 20 -> 22
- net +12VF(P): vias 7 -> 6
- added copper zone on F.Cu, net GND
Other:
- board text added: "+12V"
- board text added: "order_num"
