File: opilio_pcb/v3.1/opilio3.1.kicad_sch (KiCad schematic)
At the start: 87 parts, among them J1 Screw_Terminal_01x02, J2 Conn_01x02_Male, J3 USB_B_Micro, J4 Program, J5 Conn_01x02_Male, Q1 HSBA3048, Q2 HSBA3048, U1 AMS1117-3.3, U2 SCT51240, U3 SCT51240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

Commit message: moved opilio 3.1
Parts:
- added D10, D9: B5819W, Diode_SMD:D_SOD-123, symbol Device:D_Schottky_Small
Connections:
- net +12V: now also D9.2 (A); no longer F1.1
- net +5V: now also D10.2 (A)
- new net: D10.1 (K), D9.1 (K), F1.1
Other:
- title: Opilio 3 -> Opilio 3.1
- moved on the sheet: C1, C5, F1, FB1, U1

Commit message: almost ready for v3.1
Other:
- moved on the sheet: BL1, D2, D5, D6, D7, R16, R17, RL1
