File: opilio_pcb/v3.2/opilio3.2.kicad_sch (KiCad schematic)
At the start: 87 parts, among them J1 Screw_Terminal_01x02, J2 Conn_01x02_Male, J3 USB_B_Micro, J4 Program, J5 Conn_01x02_Male, Q1 HSBA3048, Q2 HSBA3048, U1 AMS1117-3.3, U2 SCT51240, U3 SCT51240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

Commit message: cleanup
Parts:
- R5, R7: value 220 -> 24R
Changed lines of the file:
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@@
       (effects (font (size 1.27 1.27)) (justify left))
     )
-    (property "Value" "220" (id 1) (at 189.484 64.389 90)
+    (property "Value" "24R" (id 1) (at 189.484 64.389 90)
       (effects (font (size 1.27 1.27)) (justify left))
     )
@@
       (effects (font (size 1.27 1.27)) (justify left))
     )
-    (property "Value" "220" (id 1) (at 190.246 31.75 90)
+    (property "Value" "24R" (id 1) (at 190.246 31.75 90)
       (effects (font (size 1.27 1.27)) (justify left))
     )
@@
     )
     (path "/5944723d-215f-4a6b-ab27-ec29b29bfc6b"
-      (reference "R5") (unit 1) (value "220") (footprint "Resistor_SMD:R_0603_1608Metric_Pad0.98x0.95mm_HandSolder")
+      (reference "R5") (unit 1) (value "24R") (footprint "Resistor_SMD:R_0603_1608Metric_Pad0.98x0.95mm_HandSolder")
     )
     (path "/beb113ce-d7fe-47cb-97e6-be05f9ef150e"
@@
     )
     (path "/07c1490d-aa6f-44a4-a474-a47537f0b20a"
-      (reference "R7") (unit 1) (value "220") (footprint "Resistor_SMD:R_0603_1608Metric_Pad0.98x0.95mm_HandSolder")
+      (reference "R7") (unit 1) (value "24R") (footprint "Resistor_SMD:R_0603_1608Metric_Pad0.98x0.95mm_HandSolder")
     )
     (path "/66562eec-d94a-4da6-b93e-2d8b9b62fd6f"
