File: opilio_pcb/v4.0/opilio4.0.kicad_pcb (KiCad board)
At the start: 4 copper layers, 80 x 40 mm, 81 parts, among them J1 Screw_Terminal_01x02, J2 Conn_01x02_Male, J3 USB_B_Micro, J4 Program, J5 Conn_01x02_Male, Q1 SI2306_C427393, Q2 SI2306_C427393, U1 AMS1117-3.3, U4 USBLC6-2SC6, U5 STM32F103C8T6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

Commit message: v4 almost ready
Parts:
- removed C28: 220uF, Capacitor_SMD:CP_Elec_6.3x7.7
- removed D10, D8, D9: B5819W, Diode_SMD:D_SOD-123
- removed D4: B230A-13-F, Diode_SMD:D_SMA
- removed FAN_S1: F_EN, easyedakicad:SW-SMD_L6.0-W3.3-LS8.0
- removed PUMP_S1: P_EN, easyedakicad:SW-SMD_L6.0-W3.3-LS8.0
- added BUZZER1: HNB09A03, easyeda2kicad:BUZ-TH_BD9.0-P5.00-D0.6-FD, F.Cu at (117.7, 112.5)
- added C3: 10uF, Capacitor_SMD:C_0603_1608Metric_Pad1.08x0.95mm_HandSolder, F.Cu at (162.0, 116.0)
- added C4: 22uF, Capacitor_SMD:C_1206_3216Metric_Pad1.33x1.80mm_HandSolder, F.Cu at (163.5, 129.9)
- added C7: 100nF, Capacitor_SMD:C_0603_1608Metric_Pad1.08x0.95mm_HandSolder, F.Cu at (123.5, 112.4)
- added R18: 0R, Resistor_SMD:R_0603_1608Metric_Pad0.98x0.95mm_HandSolder, F.Cu at (147.5, 126.7)
- added R2: 100R, Resistor_SMD:R_0603_1608Metric_Pad0.98x0.95mm_HandSolder, F.Cu at (130.4, 117.8)
- added R4: 10K, Resistor_SMD:R_0603_1608Metric_Pad0.98x0.95mm_HandSolder, F.Cu at (129.9, 128.8)
- added R5: 10K, Resistor_SMD:R_0603_1608Metric_Pad0.98x0.95mm_HandSolder, F.Cu at (142.9, 129.2)
- added R7: 0R, Resistor_SMD:R_0603_1608Metric_Pad0.98x0.95mm_HandSolder, F.Cu at (132.1, 124.7)
- D1: value B230A-13-F -> B230; footprint Diode_SMD:D_SMA -> Diode_SMD:D_SMB; moved to B.Cu
- D3: value B5819W -> B230; footprint Diode_SMD:D_SOD-123 -> Diode_SMD:D_SMB; moved to B.Cu
- J4: footprint Connector_PinHeader_2.54mm:PinHeader_1x04_P2.54mm_Vertical -> Connector_PinHeader_2.54mm:PinHeader_1x05_P2.54mm_Vertical
- Q1, Q2: value SI2306_C427393 -> PMV25ENEAR; footprint Package_TO_SOT_SMD:SOT-23 -> easyeda2kicad:SOT-23_L2.9-W1.3-P1.90-LS2.4-BR
- moved Q2 32.2 mm to (145.8, 129.2)
- moved D3 27.8 mm to (131.2, 132.8), turned to 0 degrees
- moved C6 26.7 mm to (134.2, 114.2)
- moved R9 24.3 mm to (147.4, 119.8), turned to 180 degrees
- moved C16 22.9 mm to (147.4, 121.5), turned to 180 degrees
- moved C17 19.7 mm to (143.6, 119.8)
- moved Q1 18.7 mm to (132.8, 128.8)
- moved C2 17.6 mm to (153.7, 134.4)
- moved R1 15.1 mm to (109.9, 111.7)
- moved D6 14.6 mm to (107.0, 129.9), turned to 90 degrees
- moved G*** 13.2 mm to (114.9, 125.2)
- moved R12 11.4 mm to (112.9, 121.2), turned to 0 degrees
- moved R10 10.9 mm to (143.6, 121.6), turned to 180 degrees
- moved Power1 10.9 mm to (117.0, 121.2)
- moved C24 10.1 mm to (147.5, 123.3)
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Connections:
- D1 pad 2: PUMP_GND -> P_GND
- D2 pad 1: PWM_READ1 -> PWM_OUT1
- D2 pad 2: PWM_OUT1 -> PWM_READ1
- D3 pad 1: FAN_GND -> +12VF(F)
- D3 pad 2: GND -> F_GND
- D5 pad 1: PWM_READ2 -> PWM_OUT2
- D5 pad 2: PWM_OUT2 -> PWM_READ2
- D6 pad 1: PWM_READ3 -> PWM_OUT3
- D6 pad 2: PWM_OUT3 -> PWM_READ3
- F1 pad 1: Net-(D10-Pad1) -> +12V
- FAN1 pad 1: FAN_GND -> F_GND
- FAN2 pad 1: FAN_GND -> F_GND
- FAN3 pad 1: FAN_GND -> F_GND
- FAN4 pad 1: FAN_GND -> F_GND
- FAN5 pad 1: FAN_GND -> F_GND
- J4 pad 2: SWCLK -> unconnected-(J4-Pad2)
- J4 pad 3: SWIO -> SWCLK
- J4 pad 4: +3.3V -> SWIO
- PUMP1 pad 1: PUMP_GND -> P_GND
- Q1 pad 1: PUMP_EN -> Net-(Q1-Pad1)
- Q1 pad 3: PUMP_GND -> F_GND
- Q2 pad 1: FAN_EN -> Net-(Q2-Pad1)
- Q2 pad 3: FAN_GND -> P_GND
- U5 pad 22: unconnected-(U5-Pad22) -> BUZZER
Routing:
- net BUZZER: track 0.00 -> 27.2 mm
- net FAN_GND: track 21.8 -> 0.00 mm, vias 5 -> 0
- net F_GND: track 0.00 -> 19.4 mm, vias 0 -> 8
- net FAN_EN: track 59.0 -> 39.6 mm
- net +5V: track 27.3 -> 8.35 mm, vias 2 -> 0
- net Net-(R2-Pad2): track 0.00 -> 12.0 mm
- net PUMP_GND: track 11.8 -> 0.00 mm
- net P_GND: track 0.00 -> 11.2 mm, vias 0 -> 1
- net Net-(D10-Pad1): track 8.86 -> 0.00 mm
- net PWM_READ2: track 49.8 -> 58.1 mm
- net PWM_OUT2: track 42.9 -> 49.9 mm, vias 2 -> 1
- net +12VF(P): track 22.4 -> 16.4 mm
- net GND: track 84.7 -> 79.2 mm, vias 33 -> 37
- net PWM_READ3: track 60.9 -> 66.2 mm
- net Net-(Q2-Pad1): track 0.00 -> 4.85 mm
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- added copper zone on B.Cu, net +3.3V
- added copper zone on F.Cu, net +3.3V
- added copper zone on F.Cu, net F_GND
- added copper zone on In1.Cu, net F_GND
- added copper zone on F.Cu, net P_GND
- removed copper zone on In1.Cu, net FAN_GND
Other:
- board text added: "Opilio V4"
- board text added: "https://github.com/mygnu/opilio-firmware"
- board text removed: "Opilio V3.3"

Commit message: ordered
Parts:
- removed U4: USBLC6-2SC6, Package_TO_SOT_SMD:SOT-23-6
- added D4: USBLC6-2SC6, easyeda2kicad:SOT-666-6_L1.6-W1.2-P0.50-LS1.6-BL, F.Cu at (168.6, 113.3)
- J1: footprint Custom:TerminalBlock_bornier-2_P5.08mm -> easyeda2kicad:CONN-TH_2P-P2.54_JL300-50002U01
- moved J1 2.21 mm to (175.6, 126.8)
- moved C13 1.62 mm to (146.7, 112.3)
- moved C14 1.48 mm to (146.7, 113.9)
- moved R6 0.11 mm to (168.3, 110.6)
Routing:
- net GND: track 79.2 -> 76.1 mm, vias 37 -> 38
- net USB_D+: track 12.4 -> 13.5 mm
- net +5V: track 8.35 -> 7.56 mm

Commit message: add tag-connect
Parts:
- removed J4: Program, Connector_PinHeader_2.54mm:PinHeader_1x05_P2.54mm_Vertical
- added SWD1: TC2030-IDC-NL_SWD, tag_connect:Tag-Connect_TC2030-IDC-NL_2x03_P1.27mm_Vertical, F.Cu at (168.1, 102.6)
- Power1: value Yellow/Green -> Green
- R16: value R165 -> 165R
Routing:
- net SWCLK: track 11.5 -> 14.7 mm
- net SWIO: track 11.8 -> 14.6 mm
- net GND: track 76.1 -> 76.9 mm, vias 38 -> 39
- net +3.3V: track 46.0 -> 46.6 mm, vias 26 -> 27
Other:
- board text removed: "3V3"
- board text removed: "SCLK"
- board text removed: "SWIO"

Commit message: update schema files
Parts:
- moved C18 0.41 mm to (148.5, 105.7)
Connections:
- C20 pad 1: Net-(C20-Pad1) -> NRST
- R14 pad 2: Net-(C20-Pad1) -> NRST
- RESET1 pad 2: Net-(C20-Pad1) -> NRST
- SWD1 pad 3: unconnected-(SWD1-Pad3) -> NRST
- U5 pad 7: Net-(C20-Pad1) -> NRST
Routing:
- net NRST: track 0.00 -> 46.6 mm
- net Net-(C20-Pad1): track 24.4 -> 0.00 mm
- net +3.3V: track 46.6 -> 45.8 mm
- net PWM_READ4: track 60.0 -> 59.3 mm
